Commit message: create bringup file to launch controllers for the gripper

File: robotiq_85_description/urdf/robotiq_85.ros2_control.xacro (robot description, xacro)
@@ -1,6 +1,9 @@
 <?xml version="1.0"?>
 <robot xmlns:xacro="http://www.ros.org/wiki/xacro">
-  <xacro:macro name="robotiq_85_ros2_control" params="name prefix
-  use_fake_hardware:=false fake_sensor_commands:=false">
+  <xacro:macro name="robotiq_85_ros2_control" params="
+  name
+  prefix
+  use_fake_hardware:=false
+  fake_sensor_commands:=false">
     <ros2_control name="${name}" type="system">
       <hardware>

File: robotiq_85_description/urdf/robotiq_85_gripper.urdf.xacro (robot description, xacro)
@@ -2,5 +2,5 @@
 <robot name="robotiq_85_gripper" xmlns:xacro="http://ros.org/wiki/xacro">
     <xacro:arg name="prefix" default="" />
-    <xacro:arg name="use_fake_hardware" default="false" />
+    <xacro:arg name="use_fake_hardware" default="true" />
     <xacro:arg name="fake_sensor_commands" default="false" />
     <xacro:include filename="$(find robotiq_85_description)/urdf/robotiq_85_gripper_macro.urdf.xacro" />
@@ -40,3 +40,12 @@
         <origin xyz="0.05 0 0.85" rpy="0 0 0"/>
     </xacro:robotiq_85_gripper>
+        <!-- ros2 control include -->
+    <xacro:include filename="$(find robotiq_85_description)/urdf/robotiq_85.ros2_control.xacro" />
+    <!-- ros2 control instance -->
+    <xacro:robotiq_85_ros2_control
+      name="Robotiq85HardwareInterface"
+      prefix="$(arg prefix)"
+      use_fake_hardware="$(arg use_fake_hardware)"
+      fake_sensor_commands="$(arg fake_sensor_commands)">
+    </xacro:robotiq_85_ros2_control>
 </robot>
