Commit message: move ros control tags to macro

File: robotiq_85_description/urdf/robotiq_85_gripper.urdf.xacro (robot description, xacro)
@@ -37,15 +37,10 @@
         </inertial>
     </link>
-    <xacro:robotiq_85_gripper prefix="" parent="gripper_root_link" >
+    <xacro:robotiq_85_gripper
+        prefix=""
+        parent="gripper_root_link"
+        use_fake_hardware="$(arg use_fake_hardware)"
+        fake_sensor_commands="$(arg fake_sensor_commands)">
         <origin xyz="0.05 0 0.85" rpy="0 0 0"/>
     </xacro:robotiq_85_gripper>
-        <!-- ros2 control include -->
-    <xacro:include filename="$(find robotiq_85_description)/urdf/robotiq_85.ros2_control.xacro" />
-    <!-- ros2 control instance -->
-    <xacro:robotiq_85_ros2_control
-      name="Robotiq85HardwareInterface"
-      prefix="$(arg prefix)"
-      use_fake_hardware="$(arg use_fake_hardware)"
-      fake_sensor_commands="$(arg fake_sensor_commands)">
-    </xacro:robotiq_85_ros2_control>
 </robot>

File: robotiq_85_description/urdf/robotiq_85_gripper_macro.urdf.xacro (robot description, xacro)
@@ -20,5 +20,14 @@
 		</gazebo>
 	</xacro:macro>
-	<xacro:macro name="robotiq_85_gripper" params="prefix parent *origin">
+	<xacro:macro name="robotiq_85_gripper" params="prefix parent use_fake_hardware fake_sensor_commands *origin">
+	<!-- ros2 control include -->
+    <xacro:include filename="$(find robotiq_85_description)/urdf/robotiq_85.ros2_control.xacro" />
+    <!-- ros2 control instance -->
+    <xacro:robotiq_85_ros2_control
+      name="Robotiq85HardwareInterface"
+      prefix="${prefix}"
+      use_fake_hardware="${use_fake_hardware}"
+      fake_sensor_commands="${fake_sensor_commands}">
+    </xacro:robotiq_85_ros2_control>
 		<joint name="${prefix}robotiq_85_base_joint" type="fixed">
 			<parent link="${parent}"/>

Commit message: add launch configuration for fake controller

File: robotiq_85_description/urdf/robotiq_85_gripper.urdf.xacro (robot description, xacro)
@@ -2,5 +2,4 @@
 <robot name="robotiq_85_gripper" xmlns:xacro="http://ros.org/wiki/xacro">
     <xacro:arg name="prefix" default="" />
-    <xacro:arg name="use_fake_hardware" default="true" />
     <xacro:arg name="fake_sensor_commands" default="false" />
     <xacro:include filename="$(find robotiq_85_description)/urdf/robotiq_85_gripper_macro.urdf.xacro" />
@@ -39,7 +38,5 @@
     <xacro:robotiq_85_gripper
         prefix=""
-        parent="gripper_root_link"
-        use_fake_hardware="$(arg use_fake_hardware)"
-        fake_sensor_commands="$(arg fake_sensor_commands)">
+        parent="gripper_root_link">
         <origin xyz="0.05 0 0.85" rpy="0 0 0"/>
     </xacro:robotiq_85_gripper>

File: robotiq_85_description/urdf/robotiq_85_gripper_macro.urdf.xacro (robot description, xacro)
@@ -20,14 +20,5 @@
 		</gazebo>
 	</xacro:macro>
-	<xacro:macro name="robotiq_85_gripper" params="prefix parent use_fake_hardware fake_sensor_commands *origin">
-	<!-- ros2 control include -->
-    <xacro:include filename="$(find robotiq_85_description)/urdf/robotiq_85.ros2_control.xacro" />
-    <!-- ros2 control instance -->
-    <xacro:robotiq_85_ros2_control
-      name="Robotiq85HardwareInterface"
-      prefix="${prefix}"
-      use_fake_hardware="${use_fake_hardware}"
-      fake_sensor_commands="${fake_sensor_commands}">
-    </xacro:robotiq_85_ros2_control>
+	<xacro:macro name="robotiq_85_gripper" params="prefix parent  *origin">
 		<joint name="${prefix}robotiq_85_base_joint" type="fixed">
 			<parent link="${parent}"/>
