Commit message: add visual links to gripper tip

File: robotiq_85_description/urdf/robotiq_85_gripper_macro.urdf.xacro (robot description, xacro)
@@ -27,9 +27,50 @@
 		</joint>
 		<link name="${prefix}robotiq_85_base_link">
-			<!-- Visual aid for grasping -->
+			<!-- Gripper body -->
+			<visual>
+				<geometry>
+					<mesh filename="package://robotiq_85_description/meshes/visual/robotiq_85_base_link.dae"/>
+				</geometry>
+			</visual>
+			<collision>
+				<geometry>
+					<mesh filename="package://robotiq_85_description/meshes/collision/robotiq_85_base_link.stl"/>
+				</geometry>
+			</collision>
+			<inertial>
+				<mass value="0.636951" />
+				<origin xyz="0.0 0.0 0.0" />
+				<inertia ixx = "0.000380" ixy = "0.000000" ixz = "0.000000"
+					iyx = "0.000000" iyy = "0.001110" iyz = "0.000000"
+					izx = "0.000000" izy = "0.000000" izz = "0.001171" />
+			</inertial>
+		</link>
+		<!-- 2 visual links to create frames for tip of the gripper and the center grasp point.-->
+		<joint name="${prefix}robotiq_85_grasp_center_joint" type="fixed">
+			<parent link="${prefix}robotiq_85_base_link"/>
+			<child link="${prefix}robotiq_85_grasp_center"/>
+			<axis xyz="0 0 1"/>
+		</joint>
+		<link name="${prefix}robotiq_85_grasp_center">
+			<visual>
+				<origin xyz="0.145 0 0" rpy="0 0 0" />
+				<geometry>
+					<sphere radius="0.005"/>
+				</geometry>
+				<material name="">
+					<color rgba="0 0.0 1.0 1.0"/>
+				</material>
+			</visual>
+		</link>
+		<joint name="${prefix}robotiq_85_grasp_tip_joint" type="fixed">
+			<parent link="${prefix}robotiq_85_grasp_center"/>
+			<child link="${prefix}robotiq_85_grasp_tip"/>
+			<axis xyz="0 0 1"/>
+		</joint>
+		<link name="${prefix}robotiq_85_grasp_tip">
 			<visual>
 				<origin xyz="0.16 0 0" rpy="0 0 0" />
 				<geometry>
-					<sphere radius="0.007"/>
+					<sphere radius="0.005"/>
 				</geometry>
 				<material name="">
@@ -37,22 +78,4 @@
 				</material>
 			</visual>
-			<!-- Gripper body -->
-			<visual>
-				<geometry>
-					<mesh filename="package://robotiq_85_description/meshes/visual/robotiq_85_base_link.dae"/>
-				</geometry>
-			</visual>
-			<collision>
-				<geometry>
-					<mesh filename="package://robotiq_85_description/meshes/collision/robotiq_85_base_link.stl"/>
-				</geometry>
-			</collision>
-			<inertial>
-				<mass value="0.636951" />
-				<origin xyz="0.0 0.0 0.0" />
-				<inertia ixx = "0.000380" ixy = "0.000000" ixz = "0.000000"
-					iyx = "0.000000" iyy = "0.001110" iyz = "0.000000"
-					izx = "0.000000" izy = "0.000000" izz = "0.001171" />
-			</inertial>
 		</link>
 		<joint name="${prefix}robotiq_85_left_knuckle_joint" type="revolute">

Commit message: change frame orientations to match tool0 from UR (Craig convention of having z-axis pointing away)

File: robotiq_85_description/urdf/robotiq_85_gripper_macro.urdf.xacro (robot description, xacro)
@@ -46,13 +46,13 @@
 			</inertial>
 		</link>
-		<!-- 2 visual links to create frames for tip of the gripper and the center grasp point.-->
+		<!-- 2 visual links to create frames for tip of the gripper and the center grasp point. Frames oriented like tool0.-->
 		<joint name="${prefix}robotiq_85_grasp_center_joint" type="fixed">
 			<parent link="${prefix}robotiq_85_base_link"/>
 			<child link="${prefix}robotiq_85_grasp_center"/>
 			<axis xyz="0 0 1"/>
+			<origin xyz="0.145 0 0" rpy="${pi/2.0} 0 ${pi/2.0}" />
 		</joint>
 		<link name="${prefix}robotiq_85_grasp_center">
 			<visual>
-				<origin xyz="0.145 0 0" rpy="0 0 0" />
 				<geometry>
 					<sphere radius="0.005"/>
@@ -67,8 +67,8 @@
 			<child link="${prefix}robotiq_85_grasp_tip"/>
 			<axis xyz="0 0 1"/>
+			<origin xyz="0 0 0.015" rpy="0 0 0" />
 		</joint>
 		<link name="${prefix}robotiq_85_grasp_tip">
 			<visual>
-				<origin xyz="0.16 0 0" rpy="0 0 0" />
 				<geometry>
 					<sphere radius="0.005"/>
